Commit message: carto

File: roverboard_cartographer/urdf/vlp16imu3d.urdf (robot description, URDF)
Before this commit: robot cartographer_backpack_3d, 3 links, 2 joints
Joints:
- removed joint vertical_vlp16_link_joint
- added joint vlp16_link_joint: type fixed, parent base_link, child velodyne, origin xyz=0.0 0. 0.05 rpy=0.0 0.0 0.0
