Commit message: adding camera

File: roverboard_description/urdf/pierrette.urdf.xacro (robot description, xacro)
@@ -1,4 +1,4 @@
 <?xml version="1.0" encoding="utf8"?>
-<robot name="jeanmarie" xmlns:xacro="http://www.ros.org/wiki/xacro">
+<robot name="pierrette" xmlns:xacro="http://www.ros.org/wiki/xacro">
   <xacro:property name="robot_name" value="pierrette" />
   <!-- Body -->
@@ -34,8 +34,11 @@
   <xacro:property name="caster_wheel_m"   value="0.25" /> <!-- wheel mass      -->
   <xacro:property name="high_definition_body_visual" value="false" />
-  <xacro:property name="high_definition_wheel_visual" value="false" />
-  <xacro:property name="high_definition_wheel_mesh" value="package://roverboard_description/meshes/hoverboard_wheel_6.5.dae" />
+  <xacro:property name="high_definition_wheel_visual" value="true" />
+  <xacro:property name="high_definition_wheel_mesh" value="package://roverboard_description/meshes/hoverboard_wheel_6.5_bis.dae" />
   <xacro:property name="high_definition_cwheel_visual" value="false" />
   <xacro:property name="high_definition_cwheel_plate_visual" value="false" />
+  <xacro:property name="use_eachine_camera" value="true" />
+  <xacro:property name="high_definition_camera_visual" value="true" />
+  <xacro:property name="use_hokuyo_lidar" value="true" />
   <xacro:include filename="$(find roverboard_description)/urdf/roverboard.urdf.xacro" />
 </robot>

File: roverboard_description/urdf/roverboard.urdf.xacro (robot description, xacro)
@@ -8,4 +8,10 @@
   <!-- Body -->
   <link name="base_link"></link>
+  <link name="base_link_footprint"></link>
+  <joint name="base_link_footprint_joint" type="fixed">
+    <origin xyz="0 0 ${-wheel_radius}" rpy="0 0 0" />
+    <parent link="base_link"/>
+    <child link="base_link_footprint" />
+  </joint>
   <link name="chassis_link">
     <visual>
@@ -42,3 +48,19 @@
   <!-- Caster -->
   <xacro:rb_caster> </xacro:rb_caster>
+  <!-- Sensors -->
+  <!-- Camera -->
+  <xacro:include filename="$(find common_robots)/urdf/sensors.urdf.xacro" />
+  <xacro:if value="${use_eachine_camera}">
+    <xacro:property name="cam_look_down_deg" value="25." />
+    <xacro:cs_camera_eachine>
+      <origin xyz="0.06 0 0.1" rpy="0 ${cam_look_down_deg/180*pi}} 0" />
+    </xacro:cs_camera_eachine>
+  </xacro:if>
+  <!-- Lidar -->
+  <xacro:if value="${use_hokuyo_lidar}">
+    <xacro:property name="laser_look_down_deg" value="5." />
+    <xacro:cs_hokuyo>
+      <origin xyz="0.04 0 0.1" rpy="0 ${laser_look_down_deg/180*pi}} 0" />
+    </xacro:cs_hokuyo>
+  </xacro:if>
 </robot>

Commit message: improving camera

File: roverboard_description/urdf/pierrette.urdf.xacro (robot description, xacro)
@@ -38,7 +38,12 @@
   <xacro:property name="high_definition_cwheel_visual" value="false" />
   <xacro:property name="high_definition_cwheel_plate_visual" value="false" />
-  <xacro:property name="use_eachine_camera" value="true" />
-  <xacro:property name="high_definition_camera_visual" value="true" />
-  <xacro:property name="use_hokuyo_lidar" value="true" />
+  <xacro:property name="use_camera" value="true" />
+  <xacro:property name="cam_hd_visual" value="true" />
+  <!-- <xacro:property name="cam_cl_to_ref_xyz" value="0.06 0 0.2" /> -->
+  <xacro:property name="cam_cl_to_ref_xyz" value="0.206   0.003  0.255" />
+  <xacro:property name="cam_look_down_deg" value="25." />
+  <!-- <xacro:property name="cam_cl_to_ref_rpy" value="0 ${cam_look_down_deg/180*pi}} 0" /> -->
+  <xacro:property name="cam_cl_to_ref_rpy" value="0.00791352  0.54611357  0.0022584" />
+  <xacro:property name="use_hokuyo_lidar" value="false" />
   <xacro:include filename="$(find roverboard_description)/urdf/roverboard.urdf.xacro" />
 </robot>

File: roverboard_description/urdf/roverboard.urdf.xacro (robot description, xacro)
@@ -51,8 +51,7 @@
   <!-- Camera -->
   <xacro:include filename="$(find common_robots)/urdf/sensors.urdf.xacro" />
-  <xacro:if value="${use_eachine_camera}">
-    <xacro:property name="cam_look_down_deg" value="25." />
-    <xacro:cs_camera_eachine>
-      <origin xyz="0.06 0 0.1" rpy="0 ${cam_look_down_deg/180*pi}} 0" />
+  <xacro:if value="${use_camera}">
+    <xacro:cs_camera_eachine cam_name="camera1" origin_ref_frame="base_link_footprint">
+      <origin xyz="${cam_cl_to_ref_xyz}" rpy="${cam_cl_to_ref_rpy}" />
     </xacro:cs_camera_eachine>
   </xacro:if>

Commit message: pierrette

File: roverboard_description/urdf/pierrette.urdf.xacro (robot description, xacro)
@@ -39,8 +39,8 @@
   <xacro:property name="high_definition_cwheel_plate_visual" value="false" />
   <xacro:property name="use_camera" value="true" />
+  <xacro:property name="cam_name" value="camera_road_front" />
   <xacro:property name="cam_hd_visual" value="true" />
-  <!-- <xacro:property name="cam_cl_to_ref_xyz" value="0.06 0 0.2" /> -->
   <xacro:property name="cam_cl_to_ref_xyz" value="0.206   0.003  0.255" />
-  <xacro:property name="cam_look_down_deg" value="25." />
+  <!-- <xacro:property name="cam_look_down_deg" value="25." /> -->
   <!-- <xacro:property name="cam_cl_to_ref_rpy" value="0 ${cam_look_down_deg/180*pi}} 0" /> -->
   <xacro:property name="cam_cl_to_ref_rpy" value="0.00791352  0.54611357  0.0022584" />
