Commit message: fixing simulation

File: roverboard_description/urdf/caroline.urdf.xacro (robot description, xacro)
@@ -1,5 +1,5 @@
 <?xml version="1.0" encoding="utf8"?>
-<robot name="jeanmarie" xmlns:xacro="http://www.ros.org/wiki/xacro">
-  <xacro:property name="robot_name" value="jeanmarie" />
+<robot name="caroline" xmlns:xacro="http://www.ros.org/wiki/xacro">
+  <xacro:property name="robot_name" value="caroline" />
   <!-- Body -->
   <xacro:property name="chassis_l"  value="0.25" />
@@ -7,5 +7,5 @@
   <xacro:property name="chassis_h"  value="0.02" />
   <xacro:property name="chassis_dz" value="0.05" />
-  <xacro:property name="chassis_dx" value="0.08" />
+  <xacro:property name="chassis_dx" value="-0.08" />
   <xacro:property name="chassis_m"  value="1.25" />
   <!-- Main wheels -->
@@ -19,5 +19,5 @@
   <xacro:property name="caster_ax1_l"     value="0.05"  /> <!-- size and location !-->
   <xacro:property name="caster_ax1_r"     value="0.01" />  <!-- of vertical axle  !-->
-  <xacro:property name="caster_ax1_dx"    value="0.18" />  <!-- wrt base_link     !-->
+  <xacro:property name="caster_ax1_dx"    value="-0.18" />  <!-- wrt base_link     !-->
   <xacro:property name="caster_ax1_dy"    value="0." />
   <xacro:property name="caster_ax1_dz"    value="0.05" />
@@ -39,9 +39,9 @@
   <xacro:property name="high_definition_cwheel_plate_visual" value="false" />
   <xacro:property name="use_camera" value="true" />
+  <xacro:property name="cam_name" value="camera_road_front" />
   <xacro:property name="cam_hd_visual" value="true" />
   <xacro:property name="cam_cl_to_ref_xyz" value="0.06483087  0.00032532  0.1591418" />
   <!-- <xacro:property name="cam_look_down_deg" value="25." /> -->
   <!-- <xacro:property name="cam_cl_to_ref_rpy" value="0 ${cam_look_down_deg/180*pi}} 0" /> -->
-  <!-- <<xacro:property name="cam_cl_to_ref_rpy" value="0.00791352  0.54611357  0.0022584" /> -->
   <xacro:property name="cam_cl_to_ref_rpy" value="0.0077082   0.47182333  0.02633946" />
   <xacro:property name="use_hokuyo_lidar" value="false" />

File: roverboard_description/urdf/roverboard.urdf.xacro (robot description, xacro)
@@ -52,5 +52,5 @@
   <xacro:include filename="$(find common_robots)/urdf/sensors.urdf.xacro" />
   <xacro:if value="${use_camera}">
-    <xacro:cs_camera_eachine cam_name="camera_road_front" origin_ref_frame="base_link_footprint">
+    <xacro:cs_camera_eachine cam_name="${cam_name}" origin_ref_frame="base_link_footprint">
       <origin xyz="${cam_cl_to_ref_xyz}" rpy="${cam_cl_to_ref_rpy}" />
     </xacro:cs_camera_eachine>

Commit message: added configurable velocity and effort limits (for simulation)

File: roverboard_description/urdf/caroline.urdf.xacro (robot description, xacro)
@@ -16,4 +16,6 @@
   <xacro:property name="wheel_joint_damping" value="0.01" />
   <xacro:property name="wheel_joint_friction" value="0.01" />
+  <xacro:property name="wheel_joint_eff_limit" value="1" />
+  <xacro:property name="wheel_joint_vel_limit" value="10" />
   <!-- Caster wheel -->
   <xacro:property name="caster_ax1_l"     value="0.05"  /> <!-- size and location !-->
@@ -45,5 +47,5 @@
   <!-- <xacro:property name="cam_cl_to_ref_rpy" value="0 ${cam_look_down_deg/180*pi}} 0" /> -->
   <xacro:property name="cam_cl_to_ref_rpy" value="0.0077082   0.47182333  0.02633946" />
-  <xacro:property name="use_hokuyo_lidar" value="false" />
+  <xacro:property name="use_hokuyo_lidar" value="true" />
   <xacro:include filename="$(find roverboard_description)/urdf/roverboard.urdf.xacro" />
 </robot>

File: roverboard_description/urdf/wheels.urdf.xacro (robot description, xacro)
@@ -35,5 +35,6 @@
       <axis xyz="0 1 0" />
       <dynamics damping="${wheel_joint_damping}" friction="${wheel_joint_friction}"/>
-      <limit effort="1" velocity="10"/>
+      <!--<limit effort="${wheel_joint_eff_limit}" velocity="${wheel_joint_vel_limit}"/>-->
+      <!--<limit effort="1" velocity="10"/>-->
     </joint>
     <transmission name="${prefix}_wheel_trans">

Commit message: start_finish

File: roverboard_description/urdf/caroline.urdf.xacro (robot description, xacro)
@@ -47,4 +47,9 @@
   <!-- <xacro:property name="cam_cl_to_ref_rpy" value="0 ${cam_look_down_deg/180*pi}} 0" /> -->
   <xacro:property name="cam_cl_to_ref_rpy" value="0.0077082   0.47182333  0.02633946" />
+  <!-- Camera 2 -->
+  <xacro:property name="use_camera2" value="true" />
+  <xacro:property name="cam2_name" value="camera_horiz_front" />
+  <xacro:property name="cam2_cl_to_ref_xyz" value="0.06483087  0.00032532  0.22" />
+  <xacro:property name="cam2_cl_to_ref_rpy" value="0.0077082   -0.1  0.02633946" />
   <xacro:property name="use_hokuyo_lidar" value="true" />
   <xacro:include filename="$(find roverboard_description)/urdf/roverboard.urdf.xacro" />

File: roverboard_description/urdf/roverboard.urdf.xacro (robot description, xacro)
@@ -56,4 +56,9 @@
     </xacro:cs_camera_eachine>
   </xacro:if>
+  <xacro:if value="${use_camera2}">
+    <xacro:cs_camera_eachine cam_name="${cam2_name}" origin_ref_frame="base_link_footprint">
+      <origin xyz="${cam2_cl_to_ref_xyz}" rpy="${cam2_cl_to_ref_rpy}" />
+    </xacro:cs_camera_eachine>
+  </xacro:if>
   <!-- Lidar -->
   <xacro:if value="${use_hokuyo_lidar}">

Commit message: fixed odometry

File: roverboard_description/urdf/caroline.urdf.xacro (robot description, xacro)
@@ -10,7 +10,7 @@
   <xacro:property name="chassis_m"  value="1.25" />
   <!-- Main wheels -->
-  <xacro:property name="wheel_radius" value="0.0375" />
+  <xacro:property name="wheel_radius" value="0.045" /> <!-- value="0.0375" /> -->
   <xacro:property name="wheel_width"  value="0.057" />
-  <xacro:property name="wheel_track"  value="0.280" />
+  <xacro:property name="wheel_track"  value="0.200" /> <!-- value="0.280" /> -->
   <xacro:property name="wheel_mass"   value="0.5" />
   <xacro:property name="wheel_joint_damping" value="0.01" />
@@ -23,5 +23,5 @@
   <xacro:property name="caster_ax1_dx"    value="-0.18" />  <!-- wrt base_link     !-->
   <xacro:property name="caster_ax1_dy"    value="0." />
-  <xacro:property name="caster_ax1_dz"    value="0.05" />
+  <xacro:property name="caster_ax1_dz"    value="0.04" />
   <xacro:property name="caster_ax1_joint_damping"    value="0.1" />
   <xacro:property name="caster_ax1_joint_friction"   value="0.01" />
@@ -41,4 +41,5 @@
   <xacro:property name="high_definition_cwheel_plate_visual" value="false" />
   <xacro:property name="use_camera" value="true" />
+  <!-- Camera 1 -->
   <xacro:property name="cam_name" value="camera_road_front" />
   <xacro:property name="cam_hd_visual" value="true" />
@@ -52,5 +53,6 @@
   <xacro:property name="cam2_cl_to_ref_xyz" value="0.06483087  0.00032532  0.22" />
   <xacro:property name="cam2_cl_to_ref_rpy" value="0.0077082   -0.1  0.02633946" />
-  <xacro:property name="use_hokuyo_lidar" value="true" />
+  <!-- Lidar -->
+  <xacro:property name="use_hokuyo_lidar" value="false" />
   <xacro:include filename="$(find roverboard_description)/urdf/roverboard.urdf.xacro" />
 </robot>

Commit message: new camera mount

File: roverboard_description/urdf/caroline.urdf.xacro (robot description, xacro)
@@ -44,8 +44,10 @@
   <xacro:property name="cam_name" value="camera_road_front" />
   <xacro:property name="cam_hd_visual" value="true" />
-  <xacro:property name="cam_cl_to_ref_xyz" value="0.06483087  0.00032532  0.1591418" />
+  <!--<xacro:property name="cam_cl_to_ref_xyz" value="0.06483087  0.00032532  0.1591418" /> -->
+  <xacro:property name="cam_cl_to_ref_xyz" value="0.03418817 -0.00488509  0.17943348" />
   <!-- <xacro:property name="cam_look_down_deg" value="25." /> -->
   <!-- <xacro:property name="cam_cl_to_ref_rpy" value="0 ${cam_look_down_deg/180*pi}} 0" /> -->
-  <xacro:property name="cam_cl_to_ref_rpy" value="0.0077082   0.47182333  0.02633946" />
+  <!--<xacro:property name="cam_cl_to_ref_rpy" value="0.0077082   0.47182333  0.02633946" /> -->
+  <xacro:property name="cam_cl_to_ref_rpy" value="0.00211058  0.64585395  0.03289786" />
   <!-- Camera 2 -->
   <xacro:property name="use_camera2" value="true" />
