Commit message: import

File: roverboard_description/urdf/roverboard.urdf.xacro (robot description, xacro)
@@ -16,16 +16,16 @@
       </xacro:if>
       <xacro:unless value="${high_definition_body_visual}">
-	<origin xyz="${chassis_dx} 0 ${chassis_dz}" rpy="0 0 0"/>
+	<origin xyz="0 0 0" rpy="0 0 0"/>
 	<geometry><box size="${chassis_l} ${chassis_w} ${chassis_h}"/></geometry>
 	<material name="light_grey" />
       </xacro:unless>
     </visual>
-    <xacro:inertial_cuboid_with_pose mass="${chassis_m}"
-				     x_length="${chassis_l}" y_length="${chassis_w}" z_length="${chassis_h}">
+    <xacro:inertial_cuboid_with_pose
+	mass="${chassis_m}" x_length="${chassis_l}" y_length="${chassis_w}" z_length="${chassis_h}">
       <origin xyz="0 0 0" rpy="0 0 0"/>
     </xacro:inertial_cuboid_with_pose>
   </link>
   <joint name="base_link_joint" type="fixed">
-    <origin xyz="0 0 0" rpy="0 0 0" />
+    <origin xyz="${chassis_dx} 0 ${chassis_dz}" rpy="0 0 0" />
     <parent link="base_link"/>
     <child link="chassis_link" />

File: roverboard_description/urdf/roverboard_1.urdf.xacro (robot description, xacro)
@@ -1,4 +1,4 @@
 <?xml version="1.0" encoding="utf8"?>
-<robot name="nono_0" xmlns:xacro="http://www.ros.org/wiki/xacro">
+<robot name="roverboard" xmlns:xacro="http://www.ros.org/wiki/xacro">
   <xacro:property name="robot_name" value="roverboard_1" />
   <xacro:property name="chassis_l"  value="0.25" />
@@ -15,5 +15,5 @@
   <xacro:property name="wheel_joint_friction" value="0.01" />
   <xacro:property name="high_definition_body_visual" value="false" />
-  <xacro:property name="high_definition_wheel_visual" value="false" />
+  <xacro:property name="high_definition_wheel_visual" value="true" />
   <xacro:include filename="$(find roverboard_description)/urdf/roverboard.urdf.xacro" />
 </robot>

File: roverboard_description/urdf/wheels.urdf.xacro (robot description, xacro)
@@ -1,7 +1,7 @@
 <?xml version="1.0"?>
-<robot name="nono" xmlns:xacro="http://www.ros.org/wiki/xacro">
+<robot name="roverboard" xmlns:xacro="http://www.ros.org/wiki/xacro">
   <!-- Wheels -->
   <xacro:macro name="wheel" params="prefix wheel_radius lr_reflect *joint_pose">
-    <xacro:property name="wheel_mesh_scale" value="${wheel_radius/0.03}" />
+    <xacro:property name="wheel_mesh_scale" value="1." />
     <link name="${prefix}_wheel_link">
       <visual>
@@ -16,5 +16,6 @@
 	  <origin xyz="0 0 0" rpy="0 0 ${lr_reflect*pi/2}"/>
           <geometry>
-	    <mesh scale="1. ${wheel_mesh_scale} ${wheel_mesh_scale}" filename="package://rosmip_description/meshes/wheel_60.dae"/>
+	    <mesh scale="1. ${wheel_mesh_scale} ${wheel_mesh_scale}"
+		  filename="package://roverboard_description/meshes/hoverboard_wheel_6.5.dae"/>
           </geometry>
 	</xacro:if>
@@ -22,7 +23,5 @@
       <collision>
         <origin xyz="0 0 0" rpy="${pi/2} 0 0"/>
-        <geometry>
-          <cylinder radius="${wheel_radius}" length="${wheel_width}"/>
-        </geometry>
+        <geometry><cylinder radius="${wheel_radius}" length="${wheel_width}"/></geometry>
       </collision>
       <xacro:inertial_cylinder_with_pose mass="${wheel_mass}" radius="${wheel_radius}" height="${wheel_width}">
@@ -31,5 +30,5 @@
     </link>
     <joint name="${prefix}_wheel_joint" type="continuous">
-      <parent link="chassis_link"/>
+      <parent link="base_link"/>
       <child link="${prefix}_wheel_link" />
       <xacro:insert_block name="joint_pose" />

Commit message: cartographer 3d running

File: roverboard_description/urdf/roverboard.urdf.xacro (robot description, xacro)
@@ -5,4 +5,5 @@
   <material name="yellow"><color rgba="0.8 0.8 0.0 0.5" /></material>
   <material name="light_grey"><color rgba="0.4 0.4 0.4 0.5" /></material>
+  <material name="tire_material"><color rgba="0 0 0.8 0.5"/></material>
   <!-- Body -->
   <link name="base_link"></link>
@@ -39,3 +40,5 @@
     <origin xyz="0 ${-(wheel_track-wheel_width)/2} 0" rpy="0 0 0" />
   </xacro:wheel>
+  <!-- Caster -->
+  <xacro:rb_caster> </xacro:rb_caster>
 </robot>

File: roverboard_description/urdf/roverboard_1.urdf.xacro (robot description, xacro)
@@ -2,18 +2,39 @@
 <robot name="roverboard" xmlns:xacro="http://www.ros.org/wiki/xacro">
   <xacro:property name="robot_name" value="roverboard_1" />
+  <!-- Body -->
   <xacro:property name="chassis_l"  value="0.25" />
   <xacro:property name="chassis_w"  value="0.22" />
-  <xacro:property name="chassis_h"  value="0.1" />
+  <xacro:property name="chassis_h"  value="0.08" />
   <xacro:property name="chassis_dz" value="0.05" />
-  <xacro:property name="chassis_dx" value="0.025" />
+  <xacro:property name="chassis_dx" value="-0.03" />
   <xacro:property name="chassis_m"  value="1.25" />
+  <!-- Main wheels -->
   <xacro:property name="wheel_radius" value="0.0825" />
   <xacro:property name="wheel_width"  value="0.05" />
-  <xacro:property name="wheel_track"  value="0.3" />
+  <xacro:property name="wheel_track"  value="0.33" />
   <xacro:property name="wheel_mass"   value="1.01" />
   <xacro:property name="wheel_joint_damping" value="0.01" />
   <xacro:property name="wheel_joint_friction" value="0.01" />
+  <!-- Caster wheel -->
+  <xacro:property name="caster_ax1_l"     value="0.05"  /> <!-- size and location !-->
+  <xacro:property name="caster_ax1_r"     value="0.01" />  <!-- of vertical axle  !-->
+  <xacro:property name="caster_ax1_dx"    value="-0.15" />  <!-- wrt base_link     !-->
+  <xacro:property name="caster_ax1_dy"    value="0." />
+  <xacro:property name="caster_ax1_dz"    value="0." />
+  <xacro:property name="caster_ax1_joint_damping"    value="0.1" />
+  <xacro:property name="caster_ax1_joint_friction"   value="0.01" />
+  <xacro:property name="caster_ax2_l"     value="0.05"/>          <!-- size and location  !-->
+  <xacro:property name="caster_ax2_r"     value="0.005"/>         <!-- of horizontal axle !-->
+  <xacro:property name="caster_ax2_loc"   value="-0.025 0 -0.05"/> <!-- wrt vert axle      !-->
+  <xacro:property name="caster_ax2_joint_damping"    value="0.1" />
+  <xacro:property name="caster_ax2_joint_friction"   value="0.01" />
+  <xacro:property name="caster_wheel_r"   value="0.035"/> <!-- Wheel diameter and hub diameter-->
+  <xacro:property name="caster_wheel_r1"  value="0.01" />
+  <xacro:property name="caster_wheel_l"   value="0.03" /> <!-- wheel thickness -->
+  <xacro:property name="caster_wheel_m"   value="0.25" /> <!-- wheel mass      -->
   <xacro:property name="high_definition_body_visual" value="false" />
   <xacro:property name="high_definition_wheel_visual" value="true" />
+  <xacro:property name="high_definition_cwheel_visual" value="true" />
+  <xacro:property name="high_definition_cwheel_plate_visual" value="false" />
   <xacro:include filename="$(find roverboard_description)/urdf/roverboard.urdf.xacro" />
 </robot>

File: roverboard_description/urdf/wheels.urdf.xacro (robot description, xacro)
@@ -1,5 +1,5 @@
 <?xml version="1.0"?>
 <robot name="roverboard" xmlns:xacro="http://www.ros.org/wiki/xacro">
-  <!-- Wheels -->
+  <!-- Main Wheels -->
   <xacro:macro name="wheel" params="prefix wheel_radius lr_reflect *joint_pose">
     <xacro:property name="wheel_mesh_scale" value="1." />
@@ -17,5 +17,5 @@
           <geometry>
 	    <mesh scale="1. ${wheel_mesh_scale} ${wheel_mesh_scale}"
-		  filename="package://roverboard_description/meshes/hoverboard_wheel_6.5.dae"/>
+		  filename="package://roverboard_description/meshes/hoverboard_wheel.dae"/>
           </geometry>
 	</xacro:if>
@@ -48,3 +48,95 @@
     </transmission>
   </xacro:macro>
+  <!--              -->
+  <!-- Caster Wheel -->
+  <!--              -->
+  <xacro:macro name="rb_caster">
+    <!-- Vertical axle -->
+    <link name="_caster_ax1_carrier_link">
+      <visual>
+        <xacro:if value="${high_definition_cwheel_plate_visual}">
+          <geometry><mesh filename="package://roverboard_description/meshes/caster.dae"/></geometry>
+        </xacro:if>
+	<xacro:unless value="${high_definition_cwheel_plate_visual}">
+	  <origin xyz="0 0 0" rpy="0 0 ${pi/2}"/>
+          <geometry><cylinder radius="${caster_ax1_r}" length="${caster_ax1_l}"/></geometry>
+          <material name="transp_green"/>
+	</xacro:unless>
+      </visual>
+      <collision>
+        <origin xyz="0 0 0" rpy="0 0 ${pi/2}"/>
+        <geometry><cylinder radius="${caster_ax1_r}" length="${caster_ax1_l}"/></geometry>
+      </collision>
+      <xacro:inertial_null/>
+    </link>
+    <joint name="$_bl_to_caster_axle_carrier_joint" type="fixed">
+      <parent link="base_link"/>
+      <child link="_caster_ax1_carrier_link"/>
+      <origin xyz="${caster_ax1_dx} ${caster_ax1_dy} ${caster_ax1_dz}"/>
+      <!--<limit effort="${caster_ax1_joint_eff_limit}" velocity="${caster_ax1_joint_vel_limit}"/>-->
+      <dynamic damping="${caster_ax1_joint_damping}" friction="{caster_ax1_joint_friction}"/>
+    </joint>
+    <!-- Horizontal axle -->
+    <link name="_caster_ax2_link">
+      <visual>
+	<origin xyz="${caster_ax2_loc}" rpy="${pi/2.} 0 0"/>
+	<geometry><cylinder radius="${caster_ax2_r}" length="${caster_ax2_l}"/></geometry>
+      </visual>
+      <xacro:inertial_null/>
+    </link>
+    <joint name="_caster_ax1_to_ax2_joint" type="continuous">
+      <parent link="_caster_ax1_carrier_link"/>
+      <child link="_caster_ax2_link"/>
+      <origin xyz="0 0 0"/>
+      <axis xyz="0 0 1"/>
+      <!--<limit effort="${caster_ax2_joint_eff_limit}" velocity="${caster_ax2_joint_vel_limit}"/>-->
+      <dynamic damping="${caster_ax2_joint_damping}" friction="{caster_ax2_joint_friction}"/>
+    </joint>
+    <transmission name="$_caster_ax1_to_ax2_trans">
+      <type>transmission_interface/SimpleTransmission</type>
+      <joint name="_caster_ax1_to_ax2_joint">
+        <hardwareInterface>hardware_interface/EffortJointInterface</hardwareInterface>
+      </joint>
+      <actuator name="_caster_ax1_act">
+        <mechanicalReduction>1</mechanicalReduction>
+      </actuator>
+    </transmission>
+    <!-- Wheel -->
+    <link name="_caster_wheel_link">
+      <visual>
+	<xacro:if value="${high_definition_cwheel_visual}">
+          <origin xyz="0 0 0" rpy="0 0 0"/>
+	  <geometry><mesh filename="package://roverboard_description/meshes/rb_caster_w_75x25.dae"/></geometry>
+        </xacro:if>
+	<xacro:unless value="${high_definition_cwheel_visual}">
+	  <origin xyz="0 0 0"/>
+          <geometry><cylinder radius="${caster_wheel_r}" length="${caster_wheel_l}"/></geometry>
+          <material name="tire_material"/>
+	</xacro:unless>
+      </visual>
+      <collision>
+	<origin xyz="0 0 0"/>
+        <geometry><cylinder radius="${caster_wheel_r}" length="${caster_wheel_l}"/></geometry>
+      </collision>
+      <xacro:inertial_hollow_tube_with_pose
+	  mass="${caster_wheel_m}" inner_rad="${caster_wheel_r1}" outer_rad="${caster_wheel_r}" height="${caster_wheel_l}">
+        <origin xyz="0 0 0" rpy="0 0 0"/>
+      </xacro:inertial_hollow_tube_with_pose>
+    </link>
+    <joint name="_caster_fork_to_wheel_joint" type="continuous">
+      <parent link="_caster_ax2_link"/>
+      <child link="_caster_wheel_link"/>
+      <origin xyz="${caster_ax2_loc}" rpy="${pi/2.} 0 0"/>
+      <axis xyz="0 0 1"/>
+    </joint>
+    <transmission name="_caster_fork_to_wheel_trans">
+      <type>transmission_interface/SimpleTransmission</type>
+      <joint name="_caster_fork_to_wheel_joint">
+        <hardwareInterface>hardware_interface/EffortJointInterface</hardwareInterface>
+      </joint>
+      <actuator name="_caster_ax2_act">
+        <mechanicalReduction>1</mechanicalReduction>
+      </actuator>
+    </transmission>
+  </xacro:macro>
 </robot>

Commit message: adding lidar to description

File: roverboard_description/urdf/roverboard.urdf.xacro (robot description, xacro)
@@ -48,5 +48,7 @@
   <!-- Caster -->
   <xacro:rb_caster> </xacro:rb_caster>
-  <!-- Sensors -->
+  <!-- ******** -->
+  <!-- Sensors  -->
+  <!-- ******** -->
   <!-- Camera -->
   <xacro:include filename="$(find common_robots)/urdf/sensors.urdf.xacro" />
@@ -63,8 +65,27 @@
   <!-- Lidar -->
   <xacro:if value="${use_hokuyo_lidar}">
-    <xacro:property name="laser_look_down_deg" value="5." />
+    <xacro:property name="laser_look_down_deg" value="0." />
     <xacro:cs_hokuyo>
-      <origin xyz="0.04 0 0.1" rpy="0 ${laser_look_down_deg/180*pi}} 0" />
+      <origin xyz="0.04 0 0.01" rpy="0 ${laser_look_down_deg/180*pi}} 0" />
     </xacro:cs_hokuyo>
   </xacro:if>
+  <xacro:if value="${use_rplidar}">
+    <xacro:cs_rplidar>
+      <origin xyz="0.04 0 0.02" rpy="0 0 0" />
+    </xacro:cs_rplidar>
+  </xacro:if>
+  <xacro:if value="${use_vlp16}">
+    <xacro:cs_vlp16>
+      <origin xyz="0. 0. 0.06" rpy="0 0 0" />
+    </xacro:cs_vlp16>
+  </xacro:if>
+  <!-- IMU -->
+  <xacro:if value="${use_imu}">
+    <link name="imu_link"/>
+    <joint name="imu_joint" type="fixed">
+      <origin xyz="0 0 0" rpy="0 0 0 " />
+      <parent link="base_link_footprint" />
+      <child link="imu_link" />
+    </joint>
+  </xacro:if>
 </robot>
