Commit message: calibrated new caroline camera

File: roverboard_description/urdf/caroline_test_amcl.urdf.xacro (robot description, xacro)
@@ -14,5 +14,9 @@
   <xacro:property name="use_camera" value="false" />
   <!-- Camera 2 -->
-  <xacro:property name="use_camera2" value="false" />
+  <!-- <xacro:property name="cam2_cl_to_ref_xyz" value="0.06483087  0.00032532  0.22" /> -->
+  <!-- <xacro:property name="cam2_cl_to_ref_rpy" value="0.0077082   -0.1  0.02633946" /> -->
+  <xacro:property name="cam2_cl_to_ref_xyz" value="0.07307767 0.01085562 0.14008273" />
+  <xacro:property name="cam2_cl_to_ref_rpy" value="-0.007879588662834792 0.05194729473215427 0.014525638137317037" />
+  <xacro:property name="use_camera2" value="true" />
   <!-- Lidar -->
   <xacro:property name="use_hokuyo_lidar" value="false" />
