Commit message: adding lidar

File: roverboard_description/urdf/caroline_defaults.urdf.xacro (robot description, xacro)
@@ -12,5 +12,5 @@
   <xacro:property name="wheel_radius" value="0.045" /> <!-- value="0.0375" /> -->
   <xacro:property name="wheel_width"  value="0.057" />
-  <xacro:property name="wheel_track"  value="0.200" /> <!-- value="0.280" /> -->
+  <xacro:property name="wheel_track"  value="0.21" /> <!-- value="0.280" /> -->
   <xacro:property name="wheel_mass"   value="0.5" />
   <xacro:property name="wheel_joint_damping" value="0.01" />
@@ -40,5 +40,5 @@
   <xacro:property name="high_definition_cwheel_visual" value="true" />
   <xacro:property name="high_definition_cwheel_plate_visual" value="false" />
-  <xacro:property name="use_camera" value="true" />
+  <xacro:property name="use_camera" value="false" />
   <!-- Camera 1 -->
   <xacro:property name="cam_name" value="camera_road_front" />
@@ -51,5 +51,5 @@
   <xacro:property name="cam_cl_to_ref_rpy" value="0.00211058  0.64585395  0.03289786" />
   <!-- Camera 2 -->
-  <xacro:property name="use_camera2" value="true" />
+  <xacro:property name="use_camera2" value="false" />
   <xacro:property name="cam2_name" value="camera_horiz_front" />
   <xacro:property name="cam2_cl_to_ref_xyz" value="0.06483087  0.00032532  0.22" />
@@ -58,6 +58,5 @@
   <xacro:property name="use_hokuyo_lidar" value="false" />
   <xacro:property name="use_rplidar" value="false" />
-  <xacro:property name="use_vlp16" value="false" />
+  <!-- IMU -->
   <xacro:property name="use_imu" value="false" />
-  <xacro:include filename="$(find roverboard_description)/urdf/roverboard.urdf.xacro" />
 </robot>

Commit message: cartographer with landmarks

File: roverboard_description/urdf/caroline_defaults.urdf.xacro (robot description, xacro)
@@ -58,4 +58,5 @@
   <xacro:property name="use_hokuyo_lidar" value="false" />
   <xacro:property name="use_rplidar" value="false" />
+  <xacro:property name="use_vlp16" value="false" />
   <!-- IMU -->
   <xacro:property name="use_imu" value="false" />

File: roverboard_description/urdf/caroline_jetson.urdf.xacro (robot description, xacro)
@@ -14,9 +14,10 @@
   <xacro:property name="use_camera" value="false" />
   <!-- Camera 2 -->
-  <xacro:property name="use_camera2" value="false" />
+  <xacro:property name="cam2_cl_to_ref_xyz" value="0.07307767 0.01085562 0.14008273" />
+  <xacro:property name="cam2_cl_to_ref_rpy" value="-0.007879588662834792 0.05194729473215427 0.014525638137317037" />
+  <xacro:property name="cam2_name" value="camera_one" />
+  <xacro:property name="use_camera2" value="true" />
   <!-- Lidar -->
-  <xacro:property name="use_hokuyo_lidar" value="false" />
   <xacro:property name="use_rplidar" value="true" />
-  <xacro:property name="use_vlp16" value="false" />
   <!-- IMU -->
   <xacro:property name="use_imu" value="false" />
